File: pcb/Shield Raspberry Pi/Shield Raspberry Pi.sch (KiCad schematic (older format))
At the start: 35 parts

Commit message: Add files via upload
Agregado de un 2n7002 y bornera + Ajuste de etiquetas
Parts:
- added J?: Conn_01x02, symbol Conn_01x02
- added Q?: 2N7002, TO_SOT_Packages_SMD:SOT-23, symbol 2N7002
- added R? (x2): R, symbol R
Connections:
- net labels added: +5V
- wire segments 114 -> 124
Changed lines of the file:
@@
 LIBS:contrib
 LIBS:valves
+LIBS:Shield Raspberry Pi-cache
 EELAYER 25 0
 EELAYER END
@@
 	4800 4800 4800 4500
 $Comp
-L +BATT #PWR?
+L +5V #PWR?
 U 1 1 5D828C15
 P 4100 4500
 F 0 "#PWR?" H 4100 4350 50  0001 C CNN
-F 1 "+BATT" H 4100 4640 50  0000 C CNN
+F 1 "+5V" H 4100 4640 50  0000 C CNN
 F 2 "" H 4100 4500 50  0001 C CNN
 F 3 "" H 4100 4500 50  0001 C CNN
@@
 	4800 6750 4800 6450
 $Comp
-L +BATT #PWR?
+L +5V #PWR?
 U 1 1 5D828C3C
 P 4100 6450
 F 0 "#PWR?" H 4100 6300 50  0001 C CNN
-F 1 "+BATT" H 4100 6590 50  0000 C CNN
+F 1 "+5V" H 4100 6590 50  0000 C CNN
 F 2 "" H 4100 6450 50  0001 C CNN
 F 3 "" H 4100 6450 50  0001 C CNN
@@
 Wire Wire Line
 	4050 1600 3950 1600
+$Comp
+L 2N7002 Q?
+U 1 1 5D8528C9
+P 6450 5550
+F 0 "Q?" H 6650 5625 50  0000 L CNN
+F 1 "2N7002" H 6650 5550 50  0000 L CNN
+F 2 "TO_SOT_Packages_SMD:SOT-23" H 6650 5475 50  0001 L CIN
+F 3 "" H 6450 5550 50  0001 L CNN
+	1    6450 5550
+	0    -1   1    0
+$EndComp
+$Comp
+L R R?
+U 1 1 5D8528CF
+P 6800 5400
+F 0 "R?" V 6880 5400 50  0000 C CNN
+F 1 "R" V 6800 5400 50  0000 C CNN
+F 2 "" V 6730 5400 50  0001 C CNN
+F 3 "" H 6800 5400 50  0001 C CNN
+	1    6800 5400
+	1    0    0    -1
+$EndComp
+$Comp
+L R R?
+U 1 1 5D8528D5
+P 6100 5400
+F 0 "R?" V 6180 5400 50  0000 C CNN
+F 1 "R" V 6100 5400 50  0000 C CNN
+F 2 "" V 6030 5400 50  0001 C CNN
+F 3 "" H 6100 5400 50  0001 C CNN
+	1    6100 5400
+	1    0    0    -1
+$EndComp
+Wire Wire Line
+	6100 5550 6100 5650
+Wire Wire Line
+	5950 5650 6250 5650
+Wire Wire Line
+	6800 5550 6800 5650
+Wire Wire Line
+	6800 5650 6650 5650
+Wire Wire Line
+	6100 4950 6100 5250
+Wire Wire Line
+	6100 5100 6450 5100
+Wire Wire Line
+	6450 5100 6450 5350
+$Comp
+L +3.3V #PWR?
+U 1 1 5D8528E2
+P 6800 4950
+F 0 "#PWR?" H 6800 4800 50  0001 C CNN
+F 1 "+3.3V" H 6800 5090 50  0000 C CNN
+F 2 "" H 6800 4950 50  0001 C CNN
+F 3 "" H 6800 4950 50  0001 C CNN
+	1    6800 4950
+	1    0    0    -1
+$EndComp
+Wire Wire Line
+	6800 5250 6800 4950
+$Comp
+L +5V #PWR?
+U 1 1 5D8528E9
+P 6100 4950
+F 0 "#PWR?" H 6100 4800 50  0001 C CNN
+F 1 "+5V" H 6100 5090 50  0000 C CNN
+F 2 "" H 6100 4950 50  0001 C CNN
+F 3 "" H 6100 4950 50  0001 C CNN
+	1    6100 4950
+	1    0    0    -1
+$EndComp
+Connection ~ 6100 5100
+$Comp
+L Conn_01x02 J?
+U 1 1 5D8528F0
+P 5750 5750
+F 0 "J?" H 5750 5850 50  0000 C CNN
+F 1 "Conn_01x02" V 5850 5700 50  0000 C CNN
+F 2 "" H 5750 5750 50  0001 C CNN
+F 3 "" H 5750 5750 50  0001 C CNN
+	1    5750 5750
+	-1   0    0    1
+$EndComp
+$Comp
+L GND #PWR?
+U 1 1 5D8528F6
+P 6100 5850
+F 0 "#PWR?" H 6100 5600 50  0001 C CNN
+F 1 "GND" H 6100 5700 50  0000 C CNN
+F 2 "" H 6100 5850 50  0001 C CNN
+F 3 "" H 6100 5850 50  0001 C CNN
+	1    6100 5850
+	1    0    0    -1
+$EndComp
+Wire Wire Line
+	6100 5850 6100 5750
+Wire Wire Line
+	6100 5750 5950 5750
+Connection ~ 6100 5650
 $EndSCHEMATC

Commit message: Add files via upload
Agregado de texto
Other:
- note added: "FALTA TERMINAR"
Changed lines of the file:
@@
 	6100 5750 5950 5750
 Connection ~ 6100 5650
+Text Notes 6700 1750 0    60   ~ 0
+FALTA TERMINAR
 $EndSCHEMATC

Commit message: Add files via upload
Parts:
- added C?: 47u, symbol CP1
- added C?: CP1, symbol CP1
- added C? (x3): C, symbol C
- added D? (x2): D_Schottky, symbol D_Schottky
- added F?: Polyfuse, symbol Polyfuse
- added J?: Jack-DC, symbol Jack-DC
- added L?: L, symbol L
- added U?: LM2596, symbol LM2596
Connections:
- wire segments 124 -> 152
Other:
- note removed: "FALTA TERMINAR"

Commit message: Add files via upload
Parts:
- added J?: Raspberry_Pi_2_3, symbol Connector:Raspberry_Pi_2_3
- C? (x2): symbol CP1 -> Device:CP1
- C? (x3): symbol C -> Device:C
- D? (x2): symbol D -> Device:D
- D? (x2): symbol D_Schottky -> Device:D_Schottky
- F?: symbol Polyfuse -> Device:Polyfuse
- J? (x3): symbol Conn_01x03 -> Shield-Raspberry-Pi-rescue:Conn_01x03
- J? (x5): symbol Conn_01x02 -> Shield-Raspberry-Pi-rescue:Conn_01x02
- J?: symbol Jack-DC -> Shield-Raspberry-Pi-rescue:Jack-DC
- K? (x2): symbol SANYOU_SRD_Form_C -> Shield-Raspberry-Pi-rescue:SANYOU_SRD_Form_C
- L?: symbol L -> Device:L
- Q? (x7): symbol 2N7002 -> Shield-Raspberry-Pi-rescue:2N7002
- R? (x19): symbol R -> Device:R
- U?: symbol MAX485E -> Shield-Raspberry-Pi-rescue:MAX485E
- U?: symbol LM2596 -> Shield-Raspberry-Pi-rescue:LM2596
Connections:
- net labels added: DE, RE, RX, TX
- wire segments 152 -> 224

Commit message: Add files via upload
Parts:
- added D?: LED1, symbol Device:LED
- added D?: LED2, symbol Device:LED
- added R? (x2): 120, symbol Shield-Raspberry-Pi-rescue:R-Device
- C?: symbol Device:CP1 -> Shield-Raspberry-Pi-rescue:CP1-Device
- C?: value CP1 -> 100u; symbol Device:CP1 -> Shield-Raspberry-Pi-rescue:CP1-Device
- C?: value C -> 10n; symbol Device:C -> Shield-Raspberry-Pi-rescue:C-Device
- C?: value C -> 100n; symbol Device:C -> Shield-Raspberry-Pi-rescue:C-Device
- C?: value C -> 1u; symbol Device:C -> Shield-Raspberry-Pi-rescue:C-Device
- D? (x2): value D -> 1N5819HW-7-F; symbol Device:D -> Shield-Raspberry-Pi-rescue:D-Device
- D?: value D_Schottky -> 1N5819HW-7-F; symbol Device:D_Schottky -> Shield-Raspberry-Pi-rescue:D_Schottky-Device
- D?: value D_Schottky -> SMBJ5.0A; symbol Device:D_Schottky -> Shield-Raspberry-Pi-rescue:D_Schottky-Device
- F?: symbol Device:Polyfuse -> Shield-Raspberry-Pi-rescue:Polyfuse-Device
- J? (x3): symbol Shield-Raspberry-Pi-rescue:Conn_01x03 -> Shield-Raspberry-Pi-rescue:Conn_01x03-Shield-Raspberry-Pi-rescue
- J? (x5): symbol Shield-Raspberry-Pi-rescue:Conn_01x02 -> Shield-Raspberry-Pi-rescue:Conn_01x02-Shield-Raspberry-Pi-rescue
- J?: symbol Shield-Raspberry-Pi-rescue:Jack-DC -> Shield-Raspberry-Pi-rescue:Jack-DC-Shield-Raspberry-Pi-rescue
- J?: symbol Connector:Raspberry_Pi_2_3 -> Shield-Raspberry-Pi-rescue:Raspberry_Pi_2_3-Connector
- K? (x2): symbol Shield-Raspberry-Pi-rescue:SANYOU_SRD_Form_C -> Shield-Raspberry-Pi-rescue:SANYOU_SRD_Form_C-Shield-Raspberry-Pi-rescue
- L?: value L -> 33uHy; symbol Device:L -> Shield-Raspberry-Pi-rescue:L-Device
- Q? (x7): symbol Shield-Raspberry-Pi-rescue:2N7002 -> Shield-Raspberry-Pi-rescue:2N7002-Shield-Raspberry-Pi-rescue
- R? (x16): value R -> 10k; symbol Device:R -> Shield-Raspberry-Pi-rescue:R-Device
- R? (x3): value R -> 120; symbol Device:R -> Shield-Raspberry-Pi-rescue:R-Device
- U?: symbol Shield-Raspberry-Pi-rescue:MAX485E -> Shield-Raspberry-Pi-rescue:MAX485E-Shield-Raspberry-Pi-rescue
- U?: value LM2596 -> LM2596 5.0; symbol Shield-Raspberry-Pi-rescue:LM2596 -> Shield-Raspberry-Pi-rescue:LM2596-Shield-Raspberry-Pi-rescue
Connections:
- net labels added: GP22, GP26
- wire segments 224 -> 245

Commit message: Add files via upload
Parts:
- removed F?: Polyfuse, symbol Shield-Raspberry-Pi-rescue:Polyfuse-Device
- C1, C5: renamed from C?; footprint (none) -> Capacitor_THT:CP_Radial_D5.0mm_P2.50mm
- C2, C3, C4: renamed from C?; footprint (none) -> Capacitor_SMD:C_0805_2012Metric
- D1, D2, D6: renamed from D?; footprint (none) -> Diode_SMD:D_SOD-123
- D3, D4: renamed from D?; footprint (none) -> LED_SMD:LED_0805_2012Metric
- D5: renamed from D?; footprint (none) -> Diode_SMD:D_SMB
- J1, J2, J3: renamed from J?; footprint (none) -> TerminalBlock:TerminalBlock_bornier-3_P5.08mm
- J10, J6, J7, J8, J9: renamed from J?; footprint (none) -> TerminalBlock:TerminalBlock_bornier-2_P5.08mm
- J4: renamed from J?; footprint (none) -> Connector_BarrelJack:BarrelJack_Horizontal
- J5: renamed from J?; footprint (none) -> Connector_PinHeader_2.54mm:PinHeader_2x20_P2.54mm_Vertical
- K1, K2: renamed from K?; footprint Relays_THT:Relay_SPDT_SANYOU_SRD_Series_Form_C -> Relay_THT:Relay_SPDT_SANYOU_SRD_Series_Form_C
- L1: renamed from L?; footprint (none) -> Inductor_THT:L_Radial_D7.0mm_P3.00mm
- Q1, Q2, Q3, Q4, Q5, Q6, Q7: renamed from Q?; footprint TO_SOT_Packages_SMD:SOT-23 -> Package_TO_SOT_SMD:SOT-23
- R1, R10, R11, R12, R13, R14, R15, R16, R17, R18, R19, R2, R20, R21, R3, R4, R5, R6, R7, R8, R9: renamed from R?; footprint (none) -> Resistor_SMD:R_0805_2012Metric
- U1: renamed from U?; footprint (none) -> Package_SO:SO-8_3.9x4.9mm_P1.27mm
- U2: renamed from U?; footprint (none) -> Package_TO_SOT_SMD:TO-263-5_TabPin3
Connections:
- net +5V: now also C2.1, C3.1, C4.1, C5.1, L1.2, U2.4 (FB)

Commit message: Add files via upload
Version completamente ruteada, faltan solo algunas leyendas
Parts:
- added D7: SS34, Diode_SMD:D_SMB, symbol Device:D
Connections:
- net at C1.1, U2.1 (VIN): now also D7.1 (K); no longer J4.1
- new net: D7.2 (A), J4.1
Changed lines of the file:
@@
 Wire Wire Line
 	4900 850  4900 800
-Wire Wire Line
-	4450 800  4900 800
 $Comp
 L Shield-Raspberry-Pi-rescue:GND-power #PWR017
@@
 	1    0    0    -1
 $EndComp
-Connection ~ 4900 800
 Wire Wire Line
 	4450 900  4500 900
@@
 Wire Wire Line
 	6150 1600 7000 1600
+$Comp
+L Device:D D7
+U 1 1 5DDA3987
+P 4700 800
+F 0 "D7" H 4700 584 50  0000 C CNN
+F 1 "SS34" H 4700 675 50  0000 C CNN
+F 2 "Diode_SMD:D_SMB" H 4700 800 50  0001 C CNN
+F 3 "~" H 4700 800 50  0001 C CNN
+	1    4700 800
+	-1   0    0    1
+$EndComp
+Wire Wire Line
+	4850 800  4900 800
+Connection ~ 4900 800
+Wire Wire Line
+	4550 800  4450 800
 $EndSCHEMATC
